Commit message: new approach simple mpc

File: xacro_to_sdf/xacro/cube.xacro (robot description, xacro)
@@ -1,27 +1,27 @@
-<?xml version="1.0" ?>
-<!-- =================================================================================== -->
-<!-- |    This document was autogenerated by xacro from xacro/cube.xacro               | -->
-<!-- |    EDITING THIS FILE BY HAND IS NOT RECOMMENDED                                 | -->
-<!-- =================================================================================== -->
-<sdf version='1.9'>
+<?xml version="1.0"?>
+<robot xmlns:xacro="http://www.ros.org/wiki/xacro">
+  <!-- Define parameters -->
+  <xacro:property name="size" value="0.1"/>
+  <xacro:property name="mass" value="0.001"/>
+  <xacro:property name="inertia" value="${(1/6) * mass * size * size}"/>
   <model name="cube">
     <link name="base_link">
       <inertial>
-        <pose>0 0 -0.05 0 0 0</pose>
-        <mass>0.001</mass>
+        <pose>0 0 ${-size/2} 0 0 0</pose>
+        <mass>${mass}</mass>
         <inertia>
-          <ixx>1.6666666666666669e-06</ixx>
+          <ixx>${inertia}</ixx>
           <ixy>0</ixy>
           <ixz>0</ixz>
-          <iyy>1.6666666666666669e-06</iyy>
+          <iyy>${inertia}</iyy>
           <iyz>0</iyz>
-          <izz>1.6666666666666669e-06</izz>
+          <izz>${inertia}</izz>
         </inertia>
       </inertial>
       <collision name="base_collision">
-        <pose>0 0 -0.05 0 0 0</pose>
+        <pose>0 0 -${size/2} 0 0 0</pose>
         <geometry>
           <box>
-            <size>0.1 0.1 0.1</size>
+            <size>${size} ${size} ${size}</size>
           </box>
         </geometry>
@@ -42,8 +42,8 @@
       </collision>
       <visual name="base_visual">
-        <pose>0 0 -0.05 0 0 0</pose>
+        <pose>0 0 -${size/2} 0 0 0</pose>
         <geometry>
           <box>
-            <size>0.1 0.1 0.1</size>
+            <size>${size} ${size} ${size}</size>
           </box>
         </geometry>
@@ -61,11 +61,4 @@
       </visual>
     </link>
-    <plugin
-      filename="gz-sim-odometry-publisher-system"
-      name="gz::sim::systems::OdometryPublisher">
-      <odom_frame>odom</odom_frame>
-      <robot_base_frame>drone_v1/cube</robot_base_frame>
-      <dimensions>3</dimensions>
-    </plugin>
   </model>
-</sdf>
+</robot>
